File: hardware/conversion_pcb/joystick.brd (EAGLE design)
At the start: 79.7 x 52.1 mm, 47 parts, among them IC1 LT1168IS8, IC2 LT1168IS8, IC3 LT1168IS8, IC4 LT1168IS8, X2 22-23-2081, X3 22-23-2101

Commit message: declutter circuit schematic
Connections:
- net N$11 renamed Z2-PRESCALE
- net N$12 renamed Z2-5V
- net N$17 renamed X-OUT
- net N$18 renamed Y-OUT
- net N$19 renamed Z-OUT
- net N$2 renamed X-PRESCALE
- net N$21 renamed X-OFFSET
- net N$22 renamed Z2-OFFSET
- net N$23 renamed Z-OFFSET
- net N$24 renamed Y-OFFSET
- net N$25 renamed Z2-OUT
- net N$3 renamed X-5V
- net N$5 renamed Y-PRESCALE
- net N$6 renamed Y-5V
- net N$8 renamed Z-PRESCALE
- net N$9 renamed Z5V
Changed lines of the file:
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@@
 <?xml version="1.0" encoding="utf-8"?>
 <!DOCTYPE eagle SYSTEM "eagle.dtd">
-<eagle version="6.6.0">
+<eagle version="7.5.0">
 <drawing>
 <settings>
@@
 <pass name="Default">
 <param name="RoutingGrid" value="50mil"/>
+<param name="AutoGrid" value="1"/>
+<param name="Efforts" value="0"/>
+<param name="TopRouterVariant" value="1"/>
 <param name="tpViaShape" value="round"/>
 <param name="PrefDir.1" value="|"/>
@@
 <wire x1="65.405" y1="19.685" x2="66.04" y2="20.32" width="0.4064" layer="1"/>
 </signal>
-<signal name="N$2">
+<signal name="X-PRESCALE">
 <contactref element="R2" pad="2"/>
 <contactref element="IC1" pad="3"/>
@@
 <wire x1="22.6945" y1="44.45" x2="17.6145" y2="49.53" width="0.6096" layer="1"/>
 </signal>
-<signal name="N$3">
+<signal name="X-5V">
 <contactref element="R2" pad="3"/>
 <wire x1="66.04" y1="40.64" x2="66.04" y2="44.45" width="0.6096" layer="1"/>
@@
 <wire x1="53.34" y1="20.955" x2="53.34" y2="20.32" width="0.4064" layer="1"/>
 </signal>
-<signal name="N$5">
+<signal name="Y-PRESCALE">
 <contactref element="R4" pad="2"/>
 <contactref element="IC2" pad="3"/>
@@
 <wire x1="19.837" y1="43.18" x2="17.6145" y2="45.4025" width="0.6096" layer="1"/>
 </signal>
-<signal name="N$6">
+<signal name="Y-5V">
 <contactref element="R4" pad="3"/>
 <contactref element="X3" pad="6"/>
@@
 <wire x1="45.085" y1="20.32" x2="48.26" y2="20.32" width="0.4064" layer="1"/>
 </signal>
-<signal name="N$8">
+<signal name="Z-PRESCALE">
 <contactref element="R6" pad="2"/>
 <contactref element="IC3" pad="3"/>
@@
 <wire x1="18.2495" y1="41.91" x2="17.6145" y2="41.275" width="0.6096" layer="1"/>
 </signal>
-<signal name="N$9">
+<signal name="Z5V">
 <contactref element="R6" pad="3"/>
 <wire x1="53.34" y1="40.64" x2="53.34" y2="44.45" width="0.6096" layer="1"/>
@@
 <wire x1="35.56" y1="20.955" x2="35.56" y2="20.32" width="0.4064" layer="1"/>
 </signal>
-<signal name="N$11">
+<signal name="Z2-PRESCALE">
 <contactref element="R8" pad="2"/>
 <contactref element="IC4" pad="3"/>
@@
 <wire x1="32.385" y1="36.195" x2="32.385" y2="38.1" width="0.6096" layer="1"/>
 </signal>
-<signal name="N$12">
+<signal name="Z2-5V">
 <contactref element="R8" pad="3"/>
 <contactref element="X2" pad="4"/>
@@
 <wire x1="39.37" y1="24.13" x2="40.005" y2="23.495" width="0.4064" layer="1"/>
 </signal>
-<signal name="N$17">
+<signal name="X-OUT">
 <contactref element="IC1" pad="6"/>
 <contactref element="X1" pad="1"/>
@@
 <wire x1="50.165" y1="15.5575" x2="49.2125" y2="16.51" width="0.4064" layer="1"/>
 </signal>
-<signal name="N$18">
+<signal name="Y-OUT">
 <contactref element="IC2" pad="6"/>
 <contactref element="X1" pad="2"/>
@@
 <wire x1="47.5742" y1="15.494" x2="50.3682" y2="12.7" width="0.4064" layer="1"/>
 </signal>
-<signal name="N$19">
+<signal name="Z-OUT">
 <contactref element="IC3" pad="6"/>
 <contactref element="R9" pad="1"/>
@@
 <wire x1="48.26" y1="10.16" x2="48.9966" y2="10.16" width="0.4064" layer="1"/>
 </signal>
-<signal name="N$21">
+<signal name="X-OFFSET">
 <contactref element="R13" pad="2"/>
 <contactref element="R14" pad="1"/>
@@
 <wire x1="19.05" y1="19.202" x2="19.05" y2="21.438" width="0.4064" layer="1"/>
 </signal>
-<signal name="N$22">
+<signal name="Z2-OFFSET">
 <contactref element="R15" pad="2"/>
 <contactref element="R16" pad="1"/>
@@
 <wire x1="11.43" y1="8.407" x2="11.43" y2="10.643" width="0.4064" layer="1"/>
 </signal>
-<signal name="N$23">
+<signal name="Z-OFFSET">
 <contactref element="R10" pad="1"/>
 <contactref element="R9" pad="2"/>
@@
 <wire x1="13.97" y1="12.217" x2="13.97" y2="14.453" width="0.4064" layer="1"/>
 </signal>
-<signal name="N$24">
+<signal name="Y-OFFSET">
 <contactref element="R11" pad="2"/>
 <contactref element="R12" pad="1"/>
@@
 <wire x1="16.51" y1="15.392" x2="16.51" y2="17.628" width="0.4064" layer="1"/>
 </signal>
-<signal name="N$25">
+<signal name="Z2-OUT">
 <contactref element="IC4" pad="6"/>
 <contactref element="R15" pad="1"/>
